File: pcb/fan_control.kicad_sch (KiCad schematic)
At the start: 6 parts, among them Q2 AO3400A

Commit message: Add temperature sensors
Parts:
- RadiatorFan2: now not fitted
Changed lines of the file:
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@@
 		(in_bom yes)
 		(on_board yes)
-		(dnp no)
+		(dnp yes)
 		(property "Reference" "RadiatorFan2"
 			(at 101.092 41.91 0)
